File: pcb/lighting_square.brd (EAGLE design)
At the start: 285 x 135 mm, 38 parts, among them IC1 ATMEGA32U2-TQFP, IC2 MC33269D 5V, J1 USB4056-03-A_REVA2, J2 BH9VPC 9V, Q1 FDN360P, Q2 16MHz

Commit message: Update lighting_square.brd
Parts:
- D1, D2, D3: value SB560 -> 1N5819; device adafruit:DO-1N4148 -> diode:DO15-12
- moved D3 7.76 mm to (67.5, 50.0), turned to 180 degrees
- moved D1 7.43 mm to (32.5, 50.0), turned to 180 degrees
- moved SV1 1.56 mm to (33.0, 17.5), turned to 270 degrees
- moved D2 0.17 mm to (50.0, 50.0), turned to 180 degrees
Routing:
- net VBUS: track 60.1 -> 84.7 mm
- net VBAT: track 31.9 -> 55.9 mm, vias 0 -> 1
- net N$15: track 31.6 -> 11.0 mm
- net N$6: track 27.8 -> 35.4 mm
- net N$17: track 14.9 -> 20.3 mm
- net 5V: track 106.1 -> 110.9 mm
- net N$2: track 14.9 -> 13.8 mm
